Commit message: Add files via upload

File: aro_sim/urdf/turtlebot3_burger2.gazebo.xacro (robot description, xacro)
@@ -1,5 +1,6 @@
 <?xml version="1.0"?>
 <robot name="turtlebot3_burger_sim" xmlns:xacro="http://ros.org/wiki/xacro">
-  <xacro:arg name="laser_visual" default="false"/>
+  <xacro:arg name="laser_visual" default="true "/>
+  <xacro:arg name="camera_visual" default="false"/>
   <xacro:arg name="imu_visual"   default="false"/>
   <gazebo reference="base_link">
@@ -47,5 +48,5 @@
       <odometryTopic>odom</odometryTopic>
       <odometryFrame>odom</odometryFrame>
-      <odometrySource>encoder</odometrySource>  <!-- world -->
+      <odometrySource>world</odometrySource>
       <publishOdomTF>true</publishOdomTF>
       <robotBaseFrame>base_footprint</robotBaseFrame>
@@ -65,16 +66,4 @@
   </gazebo>
   <gazebo>
-	<plugin name="p3d_base_controller" filename="libgazebo_ros_p3d.so">
-	  <alwaysOn>true</alwaysOn>
-	  <updateRate>50.0</updateRate>
-	  <bodyName>base_link</bodyName>
-	  <topicName>odom</topicName>
-	  <gaussianNoise>0.01</gaussianNoise>
-	  <frameName>world</frameName>
-	  <xyzOffsets>0 0 0</xyzOffsets>
-	  <rpyOffsets>0 0 0</rpyOffsets>
-	</plugin>
-  </gazebo>
-  <gazebo>
     <plugin name="imu_plugin" filename="libgazebo_ros_imu.so">
       <alwaysOn>true</alwaysOn>
@@ -84,5 +73,5 @@
       <serviceName>imu_service</serviceName>
       <gaussianNoise>0.0</gaussianNoise>
-      <updateRate>200</updateRate>
+      <updateRate>0</updateRate>
       <imu>
         <noise>
@@ -121,5 +110,5 @@
         <range>
           <min>0.120</min>
-          <max>10.0</max>  <!-- 3.5 -->
+          <max>3.5</max>
           <resolution>0.015</resolution>
         </range>
@@ -127,5 +116,5 @@
           <type>gaussian</type>
           <mean>0.0</mean>
-          <stddev>0.02</stddev> <!-- 0.01 -->
+          <stddev>0.01</stddev>
         </noise>
       </ray>
@@ -136,3 +125,46 @@
     </sensor>
   </gazebo>
+   <gazebo reference="camera_rgb_frame">
+    <sensor type="depth" name="realsense_R200">
+      <always_on>true</always_on>
+      <visualize>$(arg camera_visual)</visualize>
+      <camera>
+          <horizontal_fov>1.3439</horizontal_fov>
+          <image>
+              <width>1920</width>
+              <height>1080</height>
+              <format>R8G8B8</format>
+          </image>
+          <depth_camera></depth_camera>
+          <clip>
+              <near>0.03</near>
+              <far>100</far>
+          </clip>
+      </camera>
+      <plugin name="camera_controller" filename="libgazebo_ros_openni_kinect.so">
+        <baseline>0.2</baseline>
+        <alwaysOn>true</alwaysOn>
+        <updateRate>30.0</updateRate>
+        <cameraName>camera</cameraName>
+        <frameName>camera_rgb_optical_frame</frameName>
+        <imageTopicName>rgb/image_raw</imageTopicName>
+        <depthImageTopicName>depth/image_raw</depthImageTopicName>
+        <pointCloudTopicName>depth/points</pointCloudTopicName>
+        <cameraInfoTopicName>rgb/camera_info</cameraInfoTopicName>
+        <depthImageCameraInfoTopicName>depth/camera_info</depthImageCameraInfoTopicName>
+        <pointCloudCutoff>0.4</pointCloudCutoff>
+            <hackBaseline>0.07</hackBaseline>
+            <distortionK1>0.0</distortionK1>
+            <distortionK2>0.0</distortionK2>
+            <distortionK3>0.0</distortionK3>
+            <distortionT1>0.0</distortionT1>
+            <distortionT2>0.0</distortionT2>
+        <CxPrime>0.0</CxPrime>
+        <Cx>0.0</Cx>
+        <Cy>0.0</Cy>
+        <focalLength>0</focalLength>
+        <hackBaseline>0</hackBaseline>
+      </plugin>
+    </sensor>
+  </gazebo>
 </robot>

File: aro_sim/urdf/turtlebot3_burger_2020.gazebo.xacro (robot description, xacro)
@@ -1,5 +1,6 @@
 <?xml version="1.0"?>
-<robot name="turtlebot3_burger_sim" xmlns:xacro="http://ros.org/wiki/xacro">
+<robot name="autorace_sim" xmlns:xacro="http://ros.org/wiki/xacro">
   <xacro:arg name="laser_visual" default="false"/>
+  <xacro:arg name="camera_visual" default="false"/>
   <xacro:arg name="imu_visual"   default="false"/>
   <gazebo reference="base_link">
@@ -47,5 +48,5 @@
       <odometryTopic>odom</odometryTopic>
       <odometryFrame>odom</odometryFrame>
-      <odometrySource>encoder</odometrySource>  <!-- world -->
+      <odometrySource>world</odometrySource>
       <publishOdomTF>true</publishOdomTF>
       <robotBaseFrame>base_footprint</robotBaseFrame>
@@ -65,24 +66,11 @@
   </gazebo>
   <gazebo>
-	<plugin name="p3d_base_controller" filename="libgazebo_ros_p3d.so">
-	  <alwaysOn>true</alwaysOn>
-	  <updateRate>50.0</updateRate>
-	  <bodyName>base_link</bodyName>
-	  <topicName>odom</topicName>
-	  <gaussianNoise>0.01</gaussianNoise>
-	  <frameName>world</frameName>
-	  <xyzOffsets>0 0 0</xyzOffsets>
-	  <rpyOffsets>0 0 0</rpyOffsets>
-	</plugin>
-  </gazebo>
-  <gazebo>
     <plugin name="imu_plugin" filename="libgazebo_ros_imu.so">
       <alwaysOn>true</alwaysOn>
       <bodyName>imu_link</bodyName>
-      <frameName>imu_link</frameName>
       <topicName>imu</topicName>
       <serviceName>imu_service</serviceName>
       <gaussianNoise>0.0</gaussianNoise>
-      <updateRate>200</updateRate>
+      <updateRate>0</updateRate>
       <imu>
         <noise>
@@ -121,5 +109,5 @@
         <range>
           <min>0.120</min>
-          <max>10.0</max>  <!-- 3.5 -->
+          <max>3.5</max>
           <resolution>0.015</resolution>
         </range>
@@ -127,5 +115,5 @@
           <type>gaussian</type>
           <mean>0.0</mean>
-          <stddev>0.02</stddev> <!-- 0.01 -->
+          <stddev>0.01</stddev>
         </noise>
       </ray>
@@ -136,3 +124,47 @@
     </sensor>
   </gazebo>
+  <!--link : https://www.raspberrypi.org/documentation/hardware/camera/-->
+  <gazebo reference="camera_frame">
+    <sensor name="camera" type="wideanglecamera">
+      <always_on>true</always_on>
+      <update_rate>30</update_rate>
+      <camera>
+        <horizontal_fov>3.183</horizontal_fov>
+        <image>
+          <width>320</width>
+          <height>240</height>
+        </image>
+        <clip>
+          <near>0.1</near>
+          <far>100</far>
+        </clip>
+        <lens>
+          <type>custom</type>
+          <custom_function>
+            <c1>1.05</c1>
+            <c2>4</c2>
+            <f>1.0</f>
+            <fun>tan</fun>
+          </custom_function>
+          <scale_to_hfov>true</scale_to_hfov>
+          <cutoff_angle>3.1415</cutoff_angle>
+          <env_texture_size>512</env_texture_size>
+        </lens>
+      </camera>
+      <plugin name="camera_controller" filename="libgazebo_ros_camera.so">
+        <alwaysOn>true</alwaysOn>
+        <updateRate>30.0</updateRate>
+        <cameraName>camera</cameraName>
+        <frameName>camera_link</frameName>
+        <imageTopicName>image</imageTopicName>
+        <cameraInfoTopicName>camera_info</cameraInfoTopicName>
+        <hackBaseline>0.07</hackBaseline>
+        <distortionK1>0.0</distortionK1>
+        <distortionK2>0.0</distortionK2>
+        <distortionK3>0.0</distortionK3>
+        <distortionT1>0.0</distortionT1>
+        <distortionT2>0.0</distortionT2>
+      </plugin>
+    </sensor>
+  </gazebo>
 </robot>

File: aro_sim/urdf/turtlebot3_burger_rgbd.gazebo.xacro (robot description, xacro)
@@ -48,5 +48,5 @@
       <odometryTopic>odom</odometryTopic>
       <odometryFrame>odom</odometryFrame>
-      <odometrySource>encoder</odometrySource>  <!-- world -->
+      <odometrySource>world</odometrySource>  <!-- world(encoder)update rate 30 -->
       <publishOdomTF>true</publishOdomTF>
       <robotBaseFrame>base_footprint</robotBaseFrame>
@@ -55,5 +55,5 @@
       <publishWheelJointState>true</publishWheelJointState>
       <legacyMode>false</legacyMode>
-      <updateRate>30</updateRate>
+      <updateRate>50</updateRate>
       <leftJoint>wheel_left_joint</leftJoint>
       <rightJoint>wheel_right_joint</rightJoint>
@@ -145,5 +145,5 @@
         <baseline>0.2</baseline>
         <alwaysOn>true</alwaysOn>
-        <updateRate>30.0</updateRate>
+        <updateRate>50.0</updateRate>
         <cameraName>camera</cameraName>
         <frameName>camera_rgb_optical_frame</frameName>

File: aro_sim/urdf/turtlebot3_waffle_pi.gazebo.xacro (robot description, xacro)
@@ -1,6 +1,7 @@
 <?xml version="1.0"?>
-<robot name="turtlebot3_burger_sim" xmlns:xacro="http://ros.org/wiki/xacro">
-  <xacro:arg name="laser_visual" default="false"/>
-  <xacro:arg name="imu_visual"   default="false"/>
+<robot name="turtlebot3_waffle_pi_sim" xmlns:xacro="http://ros.org/wiki/xacro">
+  <xacro:arg name="laser_visual"  default="false"/>
+  <xacro:arg name="camera_visual" default="false"/>
+  <xacro:arg name="imu_visual"    default="false"/>
   <gazebo reference="base_link">
     <material>Gazebo/DarkGrey</material>
@@ -26,5 +27,14 @@
     <material>Gazebo/FlatBlack</material>
   </gazebo>
-  <gazebo reference="caster_back_link">
+  <gazebo reference="caster_back_right_link">
+    <mu1>0.1</mu1>
+    <mu2>0.1</mu2>
+    <kp>1000000.0</kp>
+    <kd>100.0</kd>
+    <minDepth>0.001</minDepth>
+    <maxVel>1.0</maxVel>
+    <material>Gazebo/FlatBlack</material>
+  </gazebo>
+  <gazebo reference="caster_back_left_link">
     <mu1>0.1</mu1>
     <mu2>0.1</mu2>
@@ -40,12 +50,12 @@
       <visualize>$(arg imu_visual)</visualize>
     </sensor>
-    <material>Gazebo/FlatBlack</material>
+    <material>Gazebo/Grey</material>
   </gazebo>
   <gazebo>
-    <plugin name="turtlebot3_burger_controller" filename="libgazebo_ros_diff_drive.so">
+    <plugin name="turtlebot3_waffle_pi_controller" filename="libgazebo_ros_diff_drive.so">
       <commandTopic>cmd_vel</commandTopic>
       <odometryTopic>odom</odometryTopic>
       <odometryFrame>odom</odometryFrame>
-      <odometrySource>encoder</odometrySource>  <!-- world -->
+      <odometrySource>world</odometrySource>
       <publishOdomTF>true</publishOdomTF>
       <robotBaseFrame>base_footprint</robotBaseFrame>
@@ -57,5 +67,5 @@
       <leftJoint>wheel_left_joint</leftJoint>
       <rightJoint>wheel_right_joint</rightJoint>
-      <wheelSeparation>0.160</wheelSeparation>
+      <wheelSeparation>0.287</wheelSeparation>
       <wheelDiameter>0.066</wheelDiameter>
       <wheelAcceleration>1</wheelAcceleration>
@@ -63,16 +73,4 @@
       <rosDebugLevel>na</rosDebugLevel>
     </plugin>
-  </gazebo>
-  <gazebo>
-	<plugin name="p3d_base_controller" filename="libgazebo_ros_p3d.so">
-	  <alwaysOn>true</alwaysOn>
-	  <updateRate>50.0</updateRate>
-	  <bodyName>base_link</bodyName>
-	  <topicName>odom</topicName>
-	  <gaussianNoise>0.01</gaussianNoise>
-	  <frameName>world</frameName>
-	  <xyzOffsets>0 0 0</xyzOffsets>
-	  <rpyOffsets>0 0 0</rpyOffsets>
-	</plugin>
   </gazebo>
   <gazebo>
@@ -84,5 +82,5 @@
       <serviceName>imu_service</serviceName>
       <gaussianNoise>0.0</gaussianNoise>
-      <updateRate>200</updateRate>
+      <updateRate>0</updateRate>
       <imu>
         <noise>
@@ -121,5 +119,5 @@
         <range>
           <min>0.120</min>
-          <max>10.0</max>  <!-- 3.5 -->
+          <max>3.5</max>
           <resolution>0.015</resolution>
         </range>
@@ -127,5 +125,5 @@
           <type>gaussian</type>
           <mean>0.0</mean>
-          <stddev>0.02</stddev> <!-- 0.01 -->
+          <stddev>0.01</stddev>
         </noise>
       </ray>
@@ -136,3 +134,36 @@
     </sensor>
   </gazebo>
+<!--link : https://www.raspberrypi.org/documentation/hardware/camera/-->
+  <gazebo reference="camera_rgb_frame">
+    <sensor type="camera" name="Pi Camera">
+      <always_on>true</always_on>
+      <visualize>$(arg camera_visual)</visualize>
+      <camera>
+          <horizontal_fov>1.085595</horizontal_fov>
+          <image>
+              <width>640</width>
+              <height>480</height>
+              <format>R8G8B8</format>
+          </image>
+          <clip>
+              <near>0.03</near>
+              <far>100</far>
+          </clip>
+      </camera>
+      <plugin name="camera_controller" filename="libgazebo_ros_camera.so">
+        <alwaysOn>true</alwaysOn>
+        <updateRate>30.0</updateRate>
+        <cameraName>camera</cameraName>
+        <frameName>camera_rgb_optical_frame</frameName>
+        <imageTopicName>rgb/image_raw</imageTopicName>
+        <cameraInfoTopicName>rgb/camera_info</cameraInfoTopicName>
+        <hackBaseline>0.07</hackBaseline>
+        <distortionK1>0.0</distortionK1>
+        <distortionK2>0.0</distortionK2>
+        <distortionK3>0.0</distortionK3>
+        <distortionT1>0.0</distortionT1>
+        <distortionT2>0.0</distortionT2>
+      </plugin>
+    </sensor>
+  </gazebo>
 </robot>
